File: digital lockin.brd (EAGLE design)
At the start: 76.2 x 94.9 mm, 24 parts, among them IC1 OPA2650E, IC2 LM358D, T2 NPN, U2 RASPBERRY_PICOSMD-TH, U5 TL431AIDBZR

Commit message: Final
Connections:
- removed net V+: IC1.8
- removed net V-: IC1.4
- new net N$1: C1.2, IC1.2, PD1.K, R3.1, R6.1
- new net N$11: C3.2, IC1.6, R7.1
- new net N$14: C2.2, IC1.5, R5.2
- new net N$4: C10.2, IC1.3, R9.2
- new net N$8: C3.1, IC1.7, R6.2
- net 5V: now also C8.2, IC1.8
- net ADCMID: now also C2.1, R7.2, R9.1
- net AMPOUT: now also C1.1, IC1.1, R3.2, R5.1
- net GND: now also C10.1, C8.1, IC1.4, PD1.A
Routing:
- net GND: track 0.00 -> 336.3 mm
- net 5V: track 0.00 -> 156.5 mm, vias 0 -> 3
- net ADCMID: track 0.00 -> 115.1 mm
- net AMPOUT: track 0.00 -> 95.1 mm, vias 0 -> 2
- net LEDCTRL: track 0.00 -> 67.4 mm
- net 3V3: track 0.00 -> 60.0 mm
- net ADCREF: track 0.00 -> 56.1 mm
- net N$1: track 0.00 -> 37.3 mm
- net N$11: track 0.00 -> 32.9 mm
- net N$14: track 0.00 -> 30.3 mm
- net N$4: track 0.00 -> 23.1 mm
- net N$9: track 0.00 -> 16.6 mm
- net N$8: track 0.00 -> 16.3 mm
- net N$10: track 0.00 -> 11.1 mm
- net N$20: track 0.00 -> 7.35 mm
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